File: bagel-toaster-2fet.kicad_sch (KiCad schematic)
At the start: 120 parts, among them J1 9v, J10 i2, J11 o1s, J12 o1, J13 i1, J14 i2s, J15 i1s, J16 o2s, J17 o2, J18 gnd, J19 bs, J2 gnd, J20 9v, J21 gnd, J22 9v, J23 gnd, J24 bs, J25 in, J26 out, J27 do_rtn, J28 do_snd, J29 gnd, J3 i1b, J30 gnd, J31 gnd, J32 9v, J4 o1b, J5 9v, J6 9v, J7 i2b, J8 o2b, J9 9v, Q1 J201, Q2 J113, SW1 Alpha_3PDT, SW2 Alpha_3PDT, SW3 Alpha_3PDT, SW4 3pdt, U1 4069, U2 TL074

Commit message: add sag control and reannotate
Parts:
- added sag1: 10k, Potentiometer_THT:Potentiometer_Alpha_RD901F-40-00D_Single_Vertical, symbol Device:R_Potentiometer
- renumbered C19 to C1, C16 to C10, C22 to C11, C18 to C12, C20 to C13, C12 to C14, C11 to C15, C3 to C16, C15 to C17, C5 to C18, C25 to C19, C21 to C2, C23 to C20, C24 to C21, C4 to C22, C8 to C23, C1 to C24, C6 to C25, C9 to C26, C14 to C3, C17 to C4, C7 to C5, C10 to C6, C2 to C7, C26 to C8, C13 to C9, D9 to D1, D2 to D10, D1 to D11, D14 to D13, D13 to D14, D7 to D2, D8 to D3, D6 to D4, D10 to D6, D11 to D7, D4 to D8, D3 to D9, J28 to J1, J5 to J10, J6 to J11, J30 to J12, J7 to J13, J29 to J14, J2 to J15, J8 to J16, J31 to J17, J9 to J18, J21 to J19, J24 to J2, J16 to J20, J23 to J21, J11 to J22, J18 to J23, J19 to J24, J14 to J25, J10 to J26, J17 to J27, J20 to J28, J13 to J29, J25 to J3, J15 to J30, J22 to J31, J12 to J32, J27 to J4, J3 to J5, J26 to J6, J32 to J7, J1 to J8, J4 to J9, Q2 to Q1, Q1 to Q2, R24 to R1, R22 to R10, R17 to R11, R28 to R12, R26 to R13, R27 to R14, R29 to R15, R33 to R16, R34 to R17, R2 to R18, R23 to R2, R8 to R20, R10 to R21, R14 to R22, R4 to R23, R3 to R24, R9 to R25, R6 to R26, R1 to R27, R13 to R28, R15 to R29, R21 to R3, R11 to R30, R7 to R31, R31 to R33, R30 to R34, R18 to R4, R12 to R5, R16 to R6, R5 to R7, R25 to R8, R20 to R9, SW4 to SW1, SW3 to SW2, SW2 to SW3, SW1 to SW4, U2 to U1, U1 to U2
Connections:
- net 9v: now also sag1.2, sag1.3; no longer R27.1, R31.1
- new net: R27.1, R31.1, sag1.1
Other:
- moved on the sheet: D10, J10, J11, J15, J17, J7, J8

Commit message: update annotations
Parts:
- renumbered C20 to C10, C6 to C11, C7 to C12, C5 to C13, C22 to C14, C8 to C15, C12 to C16, C24 to C17, C10 to C18, C25 to C19, C11 to C20, C13 to C21, C23 to C22, C26 to C23, C14 to C24, C9 to C25, C15 to C26, C16 to C3, C17 to C4, C3 to C5, C4 to C6, C18 to C7, C21 to C8, C19 to C9, D7 to D1, D11 to D10, D4 to D11, D5 to D12, D6 to D2, D1 to D3, D2 to D4, D3 to D5, D12 to D6, D9 to D7, D10 to D8, D8 to D9, J2 to J1, J8 to J10, J10 to J11, J7 to J12, J11 to J13, J9 to J14, J12 to J15, J15 to J16, J14 to J18, J13 to J19, J1 to J2, J16 to J20, J26 to J21, J25 to J22, J19 to J23, J27 to J24, J28 to J25, J20 to J26, J29 to J27, J30 to J28, J21 to J29, J6 to J3, J32 to J30, J22 to J32, J3 to J4, J4 to J5, J5 to J6, J24 to J7, J23 to J8, J18 to J9, R13 to R1, R4 to R10, R17 to R11, R18 to R12, R34 to R13, R24 to R14, R23 to R15, R21 to R16, R25 to R17, R22 to R18, R31 to R19, R14 to R2, R26 to R21, R5 to R22, R6 to R23, R27 to R24, R7 to R25, R10 to R26, R9 to R27, R8 to R28, R28 to R29, R2 to R3, R29 to R30, R11 to R31, R30 to R32, R32 to R33, R33 to R34, R15 to R4, R12 to R5, R1 to R6, R3 to R7, R19 to R8, R16 to R9

Commit message: 16mm pot refactor done
Parts:
- boost1, filter1, gain1, sag1, splat1, vol1, vol2: footprint Potentiometer_THT:Potentiometer_Alpha_RD901F-40-00D_Single_Vertical -> 1_mylib-footprint:pot-16mm-short-leg
Connections:
- net gainOut: now also R16.1; no longer C8.1
- net at C8.2: now also R16.2; no longer R16.1
- net at C13.2, R18.1, R22.1: now also C8.1; no longer R16.2
Other:
- moved on the sheet: C8, R16
Changed lines of the file:
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@@
 			)
 		)
-		(property "Footprint" "Potentiometer_THT:Potentiometer_Alpha_RD901F-40-00D_Single_Vertical"
+		(property "Footprint" "1_mylib-footprint:pot-16mm-short-leg"
 			(at 334.01 201.93 0)
 			(effects
@@
 			)
 		)
-		(property "Footprint" "Potentiometer_THT:Potentiometer_Alpha_RD901F-40-00D_Single_Vertical"
+		(property "Footprint" "1_mylib-footprint:pot-16mm-short-leg"
 			(at 382.27 208.28 0)
 			(effects
@@
 			)
 		)
-		(property "Footprint" "Potentiometer_THT:Potentiometer_Alpha_RD901F-40-00D_Single_Vertical"
+		(property "Footprint" "1_mylib-footprint:pot-16mm-short-leg"
 			(at 66.04 233.68 0)
 			(effects
@@
 			)
 		)
-		(property "Datasheet" "~"
+		(property "Datasheet" ""
 			(at 66.04 233.68 0)
 			(effects
@@
 			)
 		)
-		(property "Description" "Potentiometer"
+		(property "Description" ""
 			(at 66.04 233.68 0)
 			(effects
@@
 			)
 		)
-		(property "Footprint" "Potentiometer_THT:Potentiometer_Alpha_RD901F-40-00D_Single_Vertical"
+		(property "Footprint" "1_mylib-footprint:pot-16mm-short-leg"
 			(at 100.33 184.15 0)
 			(effects
@@
 	(symbol
 		(lib_id "Device:C")
-		(at 110.49 132.08 90)
+		(at 119.38 132.08 270)
 		(unit 1)
 		(exclude_from_sim no)
@@
 		(fields_autoplaced yes)
 		(property "Reference" "C8"
-			(at 110.49 124.46 90)
+			(at 119.38 124.46 90)
 			(effects
 				(font
@@
 		)
 		(property "Value" "100n"
-			(at 110.49 127 90)
+			(at 119.38 127 90)
 			(effects
 				(font
@@
 		)
 		(property "Footprint" "1_trevortjes_lib:C_CERAMIC_1x2"
-			(at 114.3 131.1148 0)
+			(at 115.57 133.0452 0)
 			(effects
 				(font
@@
 		)
 		(property "Datasheet" "~"
-			(at 110.49 132.08 0)
+			(at 119.38 132.08 0)
 			(effects
 				(font
@@
 		)
 		(property "Description" "Unpolarized capacitor"
-			(at 110.49 132.08 0)
+			(at 119.38 132.08 0)
 			(effects
 				(font
@@
 			)
 		)
-		(property "Footprint" "Potentiometer_THT:Potentiometer_Alpha_RD901F-40-00D_Single_Vertical"
+		(property "Footprint" "1_mylib-footprint:pot-16mm-short-leg"
 			(at 163.83 172.72 0)
 			(effects
@@
 	(symbol
 		(lib_id "Device:R")
-		(at 119.38 132.08 90)
+		(at 110.49 132.08 90)
 		(unit 1)
 		(exclude_from_sim no)
@@
 		(dnp no)
 		(property "Reference" "R16"
-			(at 119.38 125.73 90)
+			(at 110.49 125.73 90)
 			(effects
 				(font
@@
 		)
 		(property "Value" "10k"
-			(at 119.38 128.27 90)
+			(at 110.49 128.27 90)
 			(effects
 				(font
@@
 		)
 		(property "Footprint" "1_trevortjes_lib:R_1x4"
-			(at 119.38 133.858 90)
+			(at 110.49 133.858 90)
 			(effects
 				(font
@@
 		)
 		(property "Datasheet" "~"
-			(at 119.38 132.08 0)
+			(at 110.49 132.08 0)
 			(effects
 				(font
@@
 		)
 		(property "Description" "Resistor"
-			(at 119.38 132.08 0)
+			(at 110.49 132.08 0)
 			(effects
 				(font
@@
 			)
 		)
-		(property "Footprint" "Potentiometer_THT:Potentiometer_Alpha_RD901F-40-00D_Single_Vertical"
+		(property "Footprint" "1_mylib-footprint:pot-16mm-short-leg"
 			(at 316.23 90.17 0)
 			(effects
@@
 			)
 		)
-		(property "Footprint" "Potentiometer_THT:Potentiometer_Alpha_RD901F-40-00D_Single_Vertical"
+		(property "Footprint" "1_mylib-footprint:pot-16mm-short-leg"
 			(at 138.43 151.13 0)
 			(effects

Commit message: .
Parts:
- C15: value 100u -> 1u
Connections:
- net at C10.1, D7.1 (K), D9.2 (A)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: now also R12.1; no longer R12.2
- net at C9.1: now also R12.2; no longer R12.1
Other:
- moved on the sheet: C1, C10, C11, C12, C13, C15, C16, C18, C19, C2, C20, C21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

Commit message: one sided and smaller
Parts:
- removed D10, D8: 1N4001, Diode_THT:D_DO-41_SOD81_P7.62mm_Horizontal, symbol Diode:1N4001
- removed R11, R9: 100, 1_trevortjes_lib:R_1x4, symbol Device:R
- added D8: D_Schottky, Diode_THT:D_A-405_P7.62mm_Horizontal, symbol Device:D_Schottky
Connections:
- net 9v: now also D8.2 (A); no longer sag1.2, sag1.3
- net at C16.1: now also R26.1; no longer splat1.2
- net at C16.2: now also splat1.2; no longer R26.1
- net at U1.10 (+): now also C4.2, R8.1
- net at C3.2, R14.2: now also U1.12 (+)
- new net: D8.1 (K), sag1.2, sag1.3
Other:
- note added: "Bagel"
- note added: "Feta"
- note added: "Toaster"
- moved on the sheet: C1, C10, C11, C12, C13, C14, C15, C16, C17, C18, C19, C2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

Commit message: tidier
Connections:
- net sg1: no longer names the net of J29.1 (Pin_1), SW4.A3, SW4.C2
- net sg2: no longer names the net of J23.1 (Pin_1), SW3.A3, SW3.C2
- net sg3: no longer names the net of J8.1 (Pin_1), SW2.A1
Changed lines of the file:
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@@
-		)
-	)
-	(label "sg1"
-		(at 27.94 41.91 0)
-		(effects
-			(font
-				(size 1.27 1.27)
-			)
-			(justify left bottom)
 		)
 	)
@@
 	(label "from-drv-sw"
 		(at 86.36 44.45 0)
-		(effects
-			(font
-				(size 1.27 1.27)
-			)
-			(justify left bottom)
-		)
-	)
-	(label "sg3"
-		(at 189.23 53.34 0)
 		(effects
 			(font
@@
 		(effects
 			(font
-				(size 1.27 1.27)
-			)
-			(justify left bottom)
-		)
-	)
-	(label "sg2"
-		(at 109.22 54.61 0)
-		(effects
-			(font

Commit message: smaller
Parts:
- J1: value bs -> bx; footprint Connector_Wire:SolderWire-0.1sqmm_1x01_D0.4mm_OD1mm_Relief -> Connector_Wire:SolderWire-0.5sqmm_1x01_D0.9mm_OD2.1mm; now left out of the parts list
- J10, J11, J12, J13, J15, J16, J17, J18, J2, J3, J4, J5: footprint Connector_Wire:SolderWire-0.1sqmm_1x01_D0.4mm_OD1mm_Relief -> Connector_Wire:SolderWire-0.5sqmm_1x01_D0.9mm_OD2.1mm; now left out of the parts list
- J14: value o1b -> to; footprint Connector_Wire:SolderWire-0.1sqmm_1x01_D0.4mm_OD1mm_Relief -> Connector_Wire:SolderWire-0.5sqmm_1x01_D0.9mm_OD2.1mm; now left out of the parts list
- J19: value i2b -> fi; footprint Connector_Wire:SolderWire-0.1sqmm_1x01_D0.4mm_OD1mm_Relief -> Connector_Wire:SolderWire-0.5sqmm_1x01_D0.9mm_OD2.1mm; now left out of the parts list
- J20: value o2b -> fo; footprint Connector_Wire:SolderWire-0.1sqmm_1x01_D0.4mm_OD1mm_Relief -> Connector_Wire:SolderWire-0.5sqmm_1x01_D0.9mm_OD2.1mm; now left out of the parts list
- J6: value i1b -> bi; footprint Connector_Wire:SolderWire-0.1sqmm_1x01_D0.4mm_OD1mm_Relief -> Connector_Wire:SolderWire-0.5sqmm_1x01_D0.9mm_OD2.1mm; now left out of the parts list
- J7: value bs -> bx
Other:
- title: Toaster Feta Bagel -> Bagel Toaster Feta (Bagel)

Commit message: 1590dd
Parts:
- sag1: footprint 1_mylib-footprint:pot-16mm-short-leg -> Potentiometer_THT:Potentiometer_Alpha_RD901F-40-00D_Single_Vertical
Changed lines of the file:
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@@
 			)
 		)
-		(property "Footprint" "1_mylib-footprint:pot-16mm-short-leg"
+		(property "Footprint" "Potentiometer_THT:Potentiometer_Alpha_RD901F-40-00D_Single_Vertical"
 			(at 74.93 228.6 0)
 			(effects
@@
 			)
 		)
-		(property "Description" "sag"
+		(property "Description" ""
 			(at 74.93 228.6 0)
 			(effects
