File: bagel-toaster-2fet.kicad_sch (KiCad schematic)
At the start: 118 parts, among them J1 bx, J10 9v, J11 9v, J12 9v, J13 9v, J14 to, J15 gnd, J16 gnd, J17 gnd, J18 gnd, J19 fi, J2 do_snd, J20 fo, J21 i2, J22 i2s, J23 gnd, J24 o2, J25 9v, J26 o2s, J27 i1, J28 i1s, J29 gnd, J3 out, J30 o1, J31 9v, J32 o1s, J4 in, J5 do_rtn, J6 bi, J7 bx, J8 gnd, J9 9v, Q1 J113, Q2 J201, SW1 3pdt, SW2 Alpha_3PDT, SW3 Alpha_3PDT, SW4 Alpha_3PDT, U1 TL074, U2 4069

Commit message: fabbed
Parts:
- J21, J22, J23, J24, J25, J26, J27, J28, J29, J30, J31, J32, J7, J8, J9: footprint 1_trevortjes_lib:PAD_1_std_sqr -> Connector_Wire:SolderWire-0.5sqmm_1x01_D0.9mm_OD2.1mm; now left out of the parts list
- R21: value 10k -> 1k
Connections:
- net 9v: now also sag1.2, sag1.3; no longer D8.2 (A)
- net GND: now also U2.11; no longer U2.5
- net at U2.6: now also C18.1, R27.2
- net at D11.1 (K), R27.1: now also U2.5; no longer U2.11
- net at R19.1, R24.1: now also D8.1 (K); no longer sag1.1
- new net: D8.2 (A), sag1.1
- now unconnected: U2.10
Other:
- moved on the sheet: D8, J10, J11, J12, J13, U2C, U2E, sag1
