File: bagel-toaster-2fet.kicad_pcb (KiCad board)
At the start: 2 copper layers, 116.6 x 93.1 mm, 118 parts, among them J1 bx, J10 9v, J11 9v, J12 9v, J13 9v, J14 to, J15 gnd, J16 gnd, J17 gnd, J18 gnd, J19 fi, J2 do_snd, J20 fo, J21 i2, J22 i2s, J23 gnd, J24 o2, J25 9v, J26 o2s, J27 i1, J28 i1s, J29 gnd, J3 out, J30 o1, J31 9v, J32 o1s, J4 in, J5 do_rtn, J6 bi, J7 bx, J8 gnd, J9 9v, Q1 J113, Q2 J201, SW1 3pdt, SW2 Alpha_3PDT, SW3 Alpha_3PDT, SW4 Alpha_3PDT, U1 TL074, U2 4069

Commit message: fabbed
Parts:
- J21, J22, J23, J24, J25, J26, J27, J28, J29, J30, J31, J32, J7, J8, J9: footprint 1_trevortjes_lib:PAD_1_std_sqr -> Connector_Wire:SolderWire-0.5sqmm_1x01_D0.9mm_OD2.1mm
- R21: value 10k -> 1k
- moved J23 58.7 mm to (137.3, 71.8), turned to -90 degrees
- moved J29 52.7 mm to (99.6, 71.8)
- moved J22 52.3 mm to (137.3, 75.8), turned to -90 degrees
- moved J28 46.7 mm to (99.6, 75.8)
- moved J21 42.9 mm to (137.3, 84.0), turned to -90 degrees
- moved J26 37.6 mm to (140.8, 71.8), turned to -90 degrees
- moved J17 37.2 mm to (120.3, 65.8), turned to 180 degrees
- moved J27 37.0 mm to (99.6, 84.1)
- moved R33 36.0 mm to (145.9, 73.1), turned to -90 degrees
- moved SW2 31.3 mm to (81.1, 78.1), turned to 0 degrees
- moved SW3 30.8 mm to (157.2, 78.0), turned to 180 degrees
- moved J16 29.5 mm to (116.6, 65.8), turned to 180 degrees
- moved SW4 29.3 mm to (119.5, 78.0), turned to 180 degrees
- moved D8 29.2 mm to (130.1, 35.0), turned to 0 degrees
- moved J32 28.6 mm to (102.9, 71.8), turned to -90 degrees
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Connections:
- D8 pad 2: /9v -> Net-(D8-A)
- R19 pad 1: Net-(R19-Pad1) -> Net-(D8-K)
- R24 pad 1: Net-(R19-Pad1) -> Net-(D8-K)
- U2 pad 10: Net-(C18-Pad1) -> unconnected-(U2-Pad10)
- U2 pad 11: Net-(D11-K) -> GND
- U2 pad 5: GND -> Net-(D11-K)
- U2 pad 6: unconnected-(U2-Pad6) -> Net-(C18-Pad1)
- sag1 pad 1: Net-(R19-Pad1) -> Net-(D8-A)
- sag1 pad 2: Net-(D8-K) -> /9v
- sag1 pad 3: Net-(D8-K) -> /9v
Routing:
- net Net-(R19-Pad1): track 37.9 -> 0.00 mm
- net Net-(D8-A): track 0.00 -> 35.6 mm
- net Net-(U1B--): track 13.9 -> 37.8 mm
- net /v2: track 34.0 -> 12.9 mm
- net Net-(J28-Pin_1): track 6.10 -> 26.0 mm
- net Net-(J22-Pin_1): track 6.26 -> 26.0 mm
- net Net-(D6-K): track 24.6 -> 6.17 mm
- net Net-(J27-Pin_1): track 24.4 -> 39.5 mm
- net Net-(J1-Pin_1): track 20.2 -> 5.39 mm
- net /from-drv-sw: track 25.4 -> 39.7 mm
- net Net-(J19-Pin_1): track 19.4 -> 6.52 mm
- net /d_snd: track 16.1 -> 29.0 mm
- net Net-(Q2-G): track 18.3 -> 29.7 mm
- net /b_snd: track 59.9 -> 49.4 mm
- net /fx_in: track 9.94 -> 20.0 mm
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Other:
- board size 116.6 x 93.1 mm -> 110 x 58.8 mm
- board text added: "BB triple combo"
- board text removed: "1590xx dimensions (between screws)"
- board text removed: "Bagel Toaster Feta (Bagel)"

Commit message: oh yeah save
Parts:
- moved J27 23.9 mm to (99.3, 108.0)
- moved J28 23.9 mm to (99.3, 99.7)
- moved J29 23.9 mm to (99.3, 95.7)
- moved J30 23.9 mm to (102.6, 108.0)
- moved J31 23.9 mm to (99.3, 104.0)
- moved J32 23.9 mm to (102.6, 95.7)
- moved D6 23.9 mm to (66.8, 102.0)
- moved J22 23.9 mm to (137.0, 99.7)
- moved J9 23.9 mm to (64.8, 96.2)
- moved R33 23.9 mm to (145.6, 96.9)
- moved SW2 23.9 mm to (80.8, 102.0)
- moved D14 23.9 mm to (105.1, 101.8)
- moved J8 23.9 mm to (68.0, 107.8)
- moved R13 23.9 mm to (69.5, 104.8)
- moved SW4 23.9 mm to (119.1, 101.8)
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Other:
- board size 110 x 58.8 mm -> 110 x 82.7 mm
